Commit message: working on fixing collision avoidance

File: content/assets/urdf/franka_description/franka_panda_no_gripper_old.urdf (robot description, URDF)
Before this commit: robot panda, 13 links, 12 joints
Links:
- link panda_hand: geometry collision mesh filename=meshes/visual/hand_gripper.obj; visual mesh filename=meshes/visual/hand_gripper.obj
- link panda_link0: geometry collision mesh filename=meshes/collision/link0.obj; visual mesh filename=meshes/visual/link0.dae
- link panda_link1: geometry collision mesh filename=meshes/collision/link1.obj; visual mesh filename=meshes/visual/link1.dae
- link panda_link2: geometry collision mesh filename=meshes/collision/link2.obj; visual mesh filename=meshes/visual/link2.dae
- link panda_link3: geometry collision mesh filename=meshes/collision/link3.obj; visual mesh filename=meshes/visual/link3.dae
- link panda_link4: geometry collision mesh filename=meshes/collision/link4.obj; visual mesh filename=meshes/visual/link4.dae
- link panda_link5: geometry collision mesh filename=meshes/collision/link5.obj; visual mesh filename=meshes/visual/link5.dae
- link panda_link6: geometry collision mesh filename=meshes/collision/link6.obj; visual mesh filename=meshes/visual/link6.dae
- link panda_link7: geometry collision mesh filename=meshes/collision/link7.obj; visual mesh filename=meshes/visual/link7.dae
Joints:
- joint ee_fixed_joint: origin xyz=0.0 0. 0.0 rpy=0.0 0.0 -1.57079633 -> xyz=0.0 0. 0.0 rpy=0.0 0.0 -1.57
- joint panda_finger_joint1: origin xyz=0 0.04 0.0584 rpy=0 0 0 -> xyz=0 0 0.0584 rpy=0 0 0
- joint panda_finger_joint2: origin xyz=0 -0.04 0.0584 rpy=0 0 0 -> xyz=0 0 0.0584 rpy=0 0 0
- joint panda_fixed: origin xyz=0 0 0 rpy=0 0 0 -> xyz=0 0 0.0 rpy=0 0 0.0
- joint panda_hand_joint: axis 0 0 0 -> (none); origin xyz=0 0 0.107 rpy=0 0 -0.785398 -> xyz=0 0 0.107 rpy=0 0 -0.785398163397
- joint panda_joint2: origin xyz=0 0 0 rpy=-1.57079633 0 0 -> xyz=0 0 0 rpy=-1.57079632679 0 0
- joint panda_joint3: origin xyz=0 -0.316 0 rpy=1.57079633 0 0 -> xyz=0 -0.316 0 rpy=1.57079632679 0 0
- joint panda_joint4: origin xyz=0.0825 0 0 rpy=1.57079633 0 0 -> xyz=0.0825 0 0 rpy=1.57079632679 0 0
- joint panda_joint5: origin xyz=-0.0825 0.384 0 rpy=-1.57079633 0 0 -> xyz=-0.0825 0.384 0 rpy=-1.57079632679 0 0
- joint panda_joint6: origin xyz=0 0 0 rpy=1.57079633 0 0 -> xyz=0 0 0 rpy=1.57079632679 0 0
- joint panda_joint7: origin xyz=0.088 0 0 rpy=1.57079633 0 0 -> xyz=0.088 0 0 rpy=1.57079632679 0 0
