Commit message: ball reaching first version working with new camera setup

File: content/assets/urdf/franka_description/franka_panda_no_gripper.urdf (robot description, URDF)
Before this commit: robot panda, 11 links, 10 joints
Links:
- added link panda_leftfinger, mass 0.1; collision mesh filename=../../franka_panda_description/meshes/collision/finger.stl; visual mesh filename=../../franka_panda_description/meshes/visual/finger.dae
- added link panda_rightfinger, mass 0.1; collision mesh filename=../../franka_panda_description/meshes/collision/finger.stl; visual mesh filename=../../franka_panda_description/meshes/visual/finger.dae
- link panda_hand: mass None -> 0.73; geometry collision mesh filename=../../franka_panda_description/meshes/collision/hand.stl; visual mesh filename=../../franka_panda_description/meshes/visual/hand.dae
Joints:
- added joint panda_finger_joint1: type fixed, parent panda_hand, child panda_leftfinger, origin xyz=0 0 0.0584 rpy=0 0 0, axis 0 1 0, limit lower=0.0 upper=0.04 effort=20 velocity=0.2
- added joint panda_finger_joint2: type fixed, parent panda_hand, child panda_rightfinger, origin xyz=0 0 0.0584 rpy=0 0 0, axis 0 -1 0, limit lower=0.0 upper=0.04 effort=20 velocity=0.2, mimic joint=panda_finger_joint1

Commit message: changes to urdf and addition of other things

File: content/assets/urdf/franka_description/franka_panda_no_gripper.urdf (robot description, URDF)
Before this commit: robot panda, 13 links, 12 joints
Links:
- link panda_hand: geometry collision mesh filename=meshes/collision/hand.stl; visual mesh filename=meshes/visual/hand.dae
- link panda_leftfinger: mass 0.1 -> None; geometry collision mesh filename=meshes/collision/finger.stl; visual mesh filename=meshes/visual/finger.dae
- link panda_rightfinger: mass 0.1 -> None; geometry collision mesh filename=meshes/collision/finger.stl; visual mesh filename=meshes/visual/finger.dae

Commit message: fixed collision spheres and implemented robot_world_publisher

File: content/assets/urdf/franka_description/franka_panda_no_gripper.urdf (robot description, URDF)
Before this commit: robot panda, 13 links, 12 joints
Links:
- removed link panda_leftfinger
- removed link panda_rightfinger
Joints:
- removed joint panda_finger_joint1
- removed joint panda_finger_joint2
- joint ee_fixed_joint: origin xyz=0.0 0. 0.0 rpy=0.0 0.0 -1.57079633 -> xyz=0.0 0. 0.1 rpy=0.0 0.0 -1.57

Commit message: fixed urdfs; fixed collision sphere pub and tuned a bunch. Robot behavior looks good

File: content/assets/urdf/franka_description/franka_panda_no_gripper.urdf (robot description, URDF)
Before this commit: robot panda, 11 links, 10 joints
Links:
- added link panda_leftfinger, mass 0.1; collision mesh filename=meshes/collision/finger.stl; visual mesh filename=meshes/visual/finger.dae
- added link panda_link8
- added link panda_rightfinger, mass 0.1; collision mesh filename=meshes/collision/finger.stl; visual mesh filename=meshes/visual/finger.dae
- link panda_hand: geometry collision mesh filename=meshes/visual/hand_gripper.obj; visual mesh filename=meshes/visual/hand.dae
- link panda_link0: geometry collision mesh filename=meshes/collision/link0.obj; visual mesh filename=meshes/visual/link0.dae
- link panda_link1: mass 4.970684 -> None; geometry collision mesh filename=meshes/collision/link1.obj; visual mesh filename=meshes/visual/link1.dae
- link panda_link2: mass 0.646926 -> None; geometry collision mesh filename=meshes/collision/link2.obj; visual mesh filename=meshes/visual/link2.dae
- link panda_link3: mass 3.228604 -> None; geometry collision mesh filename=meshes/collision/link3.obj; visual mesh filename=meshes/visual/link3.dae
- link panda_link4: mass 3.587895 -> None; geometry collision mesh filename=meshes/collision/link4.obj; visual mesh filename=meshes/visual/link4.dae
- link panda_link5: mass 1.225946 -> None; geometry collision mesh filename=meshes/collision/link5.obj; visual mesh filename=meshes/visual/link5.dae
- link panda_link6: mass 1.666555 -> None; geometry collision mesh filename=meshes/collision/link6.obj; visual mesh filename=meshes/visual/link6.dae
- link panda_link7: mass 7.35522e-01 -> None; geometry collision mesh filename=meshes/collision/link7.obj; visual mesh filename=meshes/visual/link7.dae
Joints:
- added joint panda_finger_joint1: type fixed, parent panda_hand, child panda_leftfinger, origin xyz=0 0.04 0.0584 rpy=0 0 0, axis 0 1 0, limit lower=0.0 upper=0.04 effort=20 velocity=0.2
- added joint panda_finger_joint2: type fixed, parent panda_hand, child panda_rightfinger, origin xyz=0 -0.04 0.0584 rpy=0 0 0, axis 0 -1 0, limit lower=0.0 upper=0.04 effort=20 velocity=0.2
- added joint panda_joint8: type fixed, parent panda_link7, child panda_link8, origin xyz=0 0 0.107 rpy=0 0 0, axis 0 0 0
- joint panda_fixed: origin xyz=0 0 0 rpy=0 0 0 -> xyz=0 0 0.0 rpy=0 0 0.0
- joint panda_hand_joint: axis 0 0 0 -> (none); origin xyz=0 0 0.107 rpy=0 0 -0.785398 -> xyz=0 0 0 rpy=0 0 -0.785398163397; parent panda_link7 -> panda_link8
- joint panda_joint2: origin xyz=0 0 0 rpy=-1.57079633 0 0 -> xyz=0 0 0 rpy=-1.57079632679 0 0
- joint panda_joint3: origin xyz=0 -0.316 0 rpy=1.57079633 0 0 -> xyz=0 -0.316 0 rpy=1.57079632679 0 0
- joint panda_joint4: origin xyz=0.0825 0 0 rpy=1.57079633 0 0 -> xyz=0.0825 0 0 rpy=1.57079632679 0 0
- joint panda_joint5: origin xyz=-0.0825 0.384 0 rpy=-1.57079633 0 0 -> xyz=-0.0825 0.384 0 rpy=-1.57079632679 0 0
- joint panda_joint6: origin xyz=0 0 0 rpy=1.57079633 0 0 -> xyz=0 0 0 rpy=1.57079632679 0 0
- joint panda_joint7: origin xyz=0.088 0 0 rpy=1.57079633 0 0 -> xyz=0.088 0 0 rpy=1.57079632679 0 0
