Commit message: merging neel-dev changes

File: content/assets/urdf/franka_description/franka_panda_tray_test.urdf (robot description, URDF)
Before this commit: robot panda, 15 links, 14 joints
Links:
- link tray_link: geometry collision box size=0.25 0.245 0.01; visual box size=0.25 0.245 0.01
Joints:
- joint panda_tray_fixed_joint: origin xyz=-0.002 0.192 0.021 rpy=0.0 0.0 0.0 -> xyz=0.0 0.125 0.02 rpy=0.0 0.0 0.0
