Commit message: first commit for learning

File: content/assets/urdf/ball.urdf (robot description, URDF)
Before this commit: robot ball, 1 links, 0 joints
Links:
- link ball: mass 0.001 -> 0.005

File: content/assets/urdf/point_robot.urdf (robot description, URDF)
Before this commit: robot point_robot, 3 links, 2 joints
Links:
- link robot_y: mass 0.01 -> 0.1; geometry collision sphere radius=0.03; visual sphere radius=0.03
Joints:
- joint x_joint: limit lower=-0.6 upper=0.6 -> lower=-0.6 upper=0.6 effort=1 velocity=1
- joint y_joint: limit lower=-0.6 upper=0.6 -> lower=-0.6 upper=0.6 effort=1 velocity=1
