Commit message: add ball target visualization and resetting

File: content/assets/urdf/point_robot.urdf (robot description, URDF)
Before this commit: robot point_robot, 3 links, 2 joints
Links:
- link robot_y: mass None -> 0.01

Commit message: starting robot integration

File: content/assets/urdf/point_robot.urdf (robot description, URDF)
Before this commit: robot point_robot, 3 links, 2 joints
Links:
- link robot_y: mass 0.1 -> 0.01

Commit message: added torque control; must debug the reason for termination

File: content/assets/urdf/point_robot.urdf (robot description, URDF)
Before this commit: robot point_robot, 3 links, 2 joints
Links:
- link robot_y: mass 0.01 -> 1.0

Commit message: onboarding new diff_robot_mdoel, many changes to cost functions and rollouts

File: content/assets/urdf/point_robot.urdf (robot description, URDF)
Before this commit: robot point_robot, 3 links, 2 joints
Links:
- added link robot_z, mass 1.0; collision sphere radius=0.03; visual sphere radius=0.03
- link robot_y: mass 1.0 -> None; geometry 
Joints:
- added joint z_joint: type prismatic, parent robot, child robot_z, origin xyz=0 0 0.0 rpy=0 0 0, axis 0 0 1, limit lower=-0.6 upper=0.6 effort=1 velocity=1
