Commit message: temp commit for transfer to dev_neel

File: content/assets/urdf/cube.urdf (robot description, URDF)
Before this commit: robot object, 1 links, 0 joints
Links:
- link object: mass 0.5 -> 0.05

Commit message: fixing the expert

File: content/assets/urdf/cube.urdf (robot description, URDF)
Before this commit: robot object, 1 links, 0 joints
Links:
- link object: mass 0.5 -> 0.06
